File: Schematics/EPB Dongle/dongle.brd (EAGLE design)
At the start: 57.1 x 72.4 mm, 22 parts, among them IC1 MEGA48/88/168-AU, IC2 78L05Z, IC3 PCA9600SO8

Commit message: final EPB Dongle
git-svn-id: https://svn.circlemud.org/svn/rocket/trunk@836 46170a15-b891-4bf7-af97-fd374ce181e0
Routing:
- net INPUT0: track 36.5 -> 48.7 mm, vias 1 -> 0
- net DIGSEL0: track 41.4 -> 29.5 mm, vias 1 -> 2
- net GND: track 133.8 -> 122.2 mm, vias 1 -> 0
- net SEGSEL2: track 37.0 -> 26.8 mm, vias 0 -> 1
- net DIGSEL1: track 43.2 -> 37.3 mm, vias 1 -> 2
- net SPARE: track 39.9 -> 45.5 mm
- net +5V: track 67.4 -> 62.5 mm
- net BOARDSEL1: track 24.1 -> 28.8 mm, vias 1 -> 0
- net BOARDSEL2: track 31.8 -> 27.7 mm, vias 0 -> 1
- net SEGSEL1: track 19.5 -> 23.4 mm
- net INPUT1: track 36.6 -> 40.3 mm, vias 2 -> 0
- net SEGSEL0: track 18.1 -> 20.2 mm
- net SCL: track 27.0 -> 25.1 mm, vias 1 -> 2
- net BOARDSEL0: track 25.3 -> 23.5 mm
- net INPUT3: track 44.3 -> 42.8 mm, vias 1 -> 2
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
Commit message: minor edits
git-svn-id: https://svn.circlemud.org/svn/rocket/trunk@840 46170a15-b891-4bf7-af97-fd374ce181e0
Parts:
- R2, R3: value 10K -> 2K
- R6: value 10K -> 1K
- R7: value 10K -> 620
Changed lines of the file:
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@@
 <element name="PROG" library="pinhead" package="2X03" value="" x="27.432" y="30.226" rot="R180"/>
 <element name="R1" library="rcl" package="0204/5" value="10K" x="41.91" y="47.752" smashed="yes">
-<attribute name="NAME" x="36.3474" y="47.3964" size="0.9906" layer="25" ratio="10"/>
+<attribute name="NAME" x="36.6014" y="47.2694" size="0.9906" layer="25" ratio="10"/>
+<attribute name="VALUE" x="45.466" y="47.244" size="0.9906" layer="27" ratio="10"/>
 </element>
 <element name="C1" library="rcl" package="C025-025X050" value="1uF" x="21.59" y="41.402" smashed="yes" rot="R90">
@@
 <attribute name="NAME" x="47.498" y="40.894" size="1.27" layer="25" font="vector" ratio="15" rot="R90" align="center"/>
 </element>
-<element name="R2" library="rcl" package="0204/5" value="10K" x="41.91" y="45.212" smashed="yes">
-<attribute name="NAME" x="36.3474" y="44.8564" size="0.9906" layer="25" ratio="10"/>
+<element name="R2" library="rcl" package="0204/5" value="2K" x="41.91" y="45.212" smashed="yes">
+<attribute name="NAME" x="36.6014" y="44.7294" size="0.9906" layer="25" ratio="10"/>
+<attribute name="VALUE" x="45.466" y="44.704" size="0.9906" layer="27" ratio="10"/>
 </element>
-<element name="R3" library="rcl" package="0204/5" value="10K" x="41.91" y="36.322" smashed="yes" rot="R180">
-<attribute name="NAME" x="41.4274" y="34.1884" size="0.9906" layer="25" ratio="10"/>
+<element name="R3" library="rcl" package="0204/5" value="2K" x="41.91" y="36.322" smashed="yes" rot="R180">
+<attribute name="NAME" x="36.7284" y="35.8394" size="0.9906" layer="25" ratio="10"/>
+<attribute name="VALUE" x="45.8724" y="35.7886" size="0.9906" layer="27" ratio="10"/>
 </element>
 <element name="IC2" library="linear" package="TO92" value="78L05Z" x="40.894" y="30.226" smashed="yes" rot="R90">
@@
 <attribute name="NAME" x="48.006" y="28.956" size="1.27" layer="25" ratio="10" rot="R90"/>
 </element>
-<element name="R6" library="rcl" package="0204/5" value="10K" x="52.07" y="31.75" smashed="yes" rot="R180">
-<attribute name="NAME" x="51.308" y="29.6164" size="0.9906" layer="25" ratio="10"/>
+<element name="R6" library="rcl" package="0204/5" value="1K" x="52.07" y="31.75" smashed="yes" rot="R180">
+<attribute name="NAME" x="49.784" y="29.718" size="0.9906" layer="25" ratio="10"/>
+<attribute name="VALUE" x="52.4764" y="29.6926" size="0.9906" layer="27" ratio="10"/>
 </element>
-<element name="R7" library="rcl" package="0204/5" value="10K" x="52.07" y="44.704" smashed="yes" rot="R180">
-<attribute name="NAME" x="51.308" y="45.8724" size="0.9906" layer="25" ratio="10"/>
+<element name="R7" library="rcl" package="0204/5" value="620" x="52.07" y="44.704" smashed="yes" rot="R180">
+<attribute name="NAME" x="50.038" y="45.72" size="0.9906" layer="25" ratio="10"/>
+<attribute name="VALUE" x="52.578" y="45.72" size="0.9906" layer="27" ratio="10"/>
 </element>
 <element name="12V" library="led" package="LED3MM" value="" x="52.07" y="35.56" smashed="yes" rot="R180">
