File: Schematics/EPB Dongle/dongle.sch (EAGLE design)
At the start: 19 parts, among them IC1 MEGA48/88/168-AU, IC2 78L05Z, IC3 PCA9600SO8

Commit message: minor edits
git-svn-id: https://svn.circlemud.org/svn/rocket/trunk@840 46170a15-b891-4bf7-af97-fd374ce181e0
Parts:
- R2, R3: value 10K -> 2K
- R6: value 10K -> 1K
- R7: value 10K -> 620
Changed lines of the file:
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@@
 <part name="IC3" library="4534_I2C2" deviceset="PCA9600" device="SO8"/>
 <part name="GND3" library="supply1" deviceset="GND" device=""/>
-<part name="R2" library="rcl" deviceset="R-US_" device="0204/5" value="10K"/>
-<part name="R3" library="rcl" deviceset="R-US_" device="0204/5" value="10K"/>
+<part name="R2" library="rcl" deviceset="R-US_" device="0204/5" value="2K"/>
+<part name="R3" library="rcl" deviceset="R-US_" device="0204/5" value="2K"/>
 <part name="P+3" library="supply1" deviceset="+5V" device=""/>
 <part name="P+4" library="supply1" deviceset="+5V" device=""/>
@@
 <part name="P+10" library="supply1" deviceset="+12V" device=""/>
 <part name="P+11" library="supply1" deviceset="+5V" device=""/>
-<part name="R6" library="rcl" deviceset="R-US_" device="0204/5" value="10K"/>
-<part name="R7" library="rcl" deviceset="R-US_" device="0204/5" value="10K"/>
+<part name="R6" library="rcl" deviceset="R-US_" device="0204/5" value="1K"/>
+<part name="R7" library="rcl" deviceset="R-US_" device="0204/5" value="620"/>
 <part name="GND5" library="supply1" deviceset="GND" device=""/>
 <part name="GND6" library="supply1" deviceset="GND" device=""/>
