File: Schematics/Ikea Lighting System/Rev B/lightcontrol.brd (EAGLE design)
At the start: 60.8 x 30 mm, 21 parts, among them IC1 7803, Q1 BS170, Q2 BS170, Q3 BS170, Q4 DMP2035U, U1 V7805-1000R, U2 STM32F303K8T6

Commit message: Minor update to Ikea Lighting Controller Rev B
Parts:
- U$1: value SAMTEC-TFM-105-01-X-DJ -> CORTEX_HEADERJ; device SAMTEC-TFM-105-01-X-D:SAMTEC-TFM-105-01-X-D -> Lectrobox:CORTEX_HEADER
- moved U$1 1.31 mm to (54.2, 4.19)
- moved SERIAL 0.51 mm to (43.4, 3.30)
Connections:
- net VCC: now also U$1.1
Routing:
- net VCC: track 25.2 -> 46.2 mm
- net RESET: track 23.4 -> 21.9 mm
- net SWIO: track 11.1 -> 9.97 mm
- net SWCLK: track 11.3 -> 10.2 mm
- net RX: track 9.81 -> 9.15 mm
Other:
- board text added: "TX RX GND"
