File: Schematics/Ikea Lighting System/Rev B/lightcontrol.sch (EAGLE design)
At the start: 21 parts, among them IC1 7803, Q1 BS170, Q2 BS170, Q3 BS170, Q4 DMP2035U, U1 V7805-1000R, U2 STM32F303K8T6

Commit message: Minor update to Ikea Lighting Controller Rev B
Parts:
- U$1: value SAMTEC-TFM-105-01-X-DJ -> CORTEX_HEADERJ; device SAMTEC-TFM-105-01-X-D:SAMTEC-TFM-105-01-X-DJ -> Lectrobox:CORTEX_HEADERJ
Connections:
- net VCC: now also U$1.1
Changed lines of the file:
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@@
 <layer number="106" name="bPlate" color="7" fill="1" visible="no" active="yes"/>
 <layer number="107" name="Crop" color="7" fill="1" visible="no" active="yes"/>
+<layer number="108" name="tplace-old" color="10" fill="1" visible="yes" active="yes"/>
+<layer number="109" name="ref-old" color="11" fill="1" visible="yes" active="yes"/>
 <layer number="116" name="Patch_BOT" color="9" fill="4" visible="no" active="yes"/>
 <layer number="121" name="_tsilk" color="7" fill="1" visible="no" active="yes"/>
@@
 <layer number="144" name="Drill_legend" color="7" fill="1" visible="no" active="yes"/>
 <layer number="151" name="HeatSink" color="7" fill="1" visible="no" active="yes"/>
+<layer number="199" name="Contour" color="7" fill="1" visible="yes" active="yes"/>
 <layer number="200" name="200bmp" color="1" fill="10" visible="no" active="no"/>
 <layer number="201" name="201bmp" color="2" fill="10" visible="no" active="yes"/>
@@
 <part name="C2" library="rcl" deviceset="C-US" device="050-035X075" value="10uF"/>
 <part name="IC1" library="linear" library_urn="urn:adsk.eagle:library:262" deviceset="78*" device="Z" package3d_urn="urn:adsk.eagle:package:16416/2" technology="L05" value="7803"/>
-<part name="U$1" library="SAMTEC-TFM-105-01-X-D" deviceset="SAMTEC-TFM-105-01-X-D" device="J"/>
+<part name="U$1" library="Lectrobox" deviceset="CORTEX_HEADER" device="J"/>
 <part name="FRAME2" library="frames" library_urn="urn:adsk.eagle:library:229" deviceset="LETTER_L" device=""/>
 <part name="GND2" library="supply1" deviceset="GND" device=""/>
@@
 <part name="GND6" library="supply1" deviceset="GND" device=""/>
 <part name="U1" library="V7805-1000R" deviceset="V7805-1000R" device=""/>
+<part name="P+4" library="supply1" library_urn="urn:adsk.eagle:library:371" deviceset="VCC" device=""/>
 </parts>
 <sheets>
@@
 <attribute name="VALUE" x="149.8026" y="88.8617" size="1.27478125" layer="95"/>
 </instance>
+<instance part="P+4" gate="VCC" x="53.34" y="109.22" smashed="yes">
+<attribute name="VALUE" x="50.8" y="106.68" size="1.778" layer="96" rot="R90"/>
+</instance>
 </instances>
 <busses>
@@
 <wire x1="233.68" y1="101.6" x2="233.68" y2="106.68" width="0.1524" layer="91"/>
 </segment>
-</net>
+<segment>
+<pinref part="P+4" gate="VCC" pin="VCC"/>
+<wire x1="53.34" y1="106.68" x2="53.34" y2="99.06" width="0.1524" layer="91"/>
+<pinref part="U$1" gate="A" pin="1"/>
+<wire x1="53.34" y1="99.06" x2="60.96" y2="99.06" width="0.1524" layer="91"/>
+</segment>
+</net>
